Commit message: fix: harden phase-0 integration

File: ros2/pybullet_ros/urdf/drone.urdf.xacro (robot description, xacro)
@@ -1,17 +1,10 @@
 <?xml version="1.0"?>
 <robot xmlns:xacro="http://ros.org/wiki/xacro">
-  <xacro:macro name="drone_macro" params="suffix parent x_dist y_dist z_dist radius">
-    <link name="base_${suffix}"/>
+  <xacro:macro name="drone_macro" params="suffix parent">
     <link name="baselink_${suffix}"/>
     <link name="sensor_${suffix}"/>
-    <link name="odom_${suffix}"/>
-    <joint name="base_${suffix}_joint" type="fixed">
-      <origin rpy="0 0 ${radians(radius)}" xyz="${x_dist} ${y_dist} ${z_dist}"/>
-      <parent link="${parent}"/>
-      <child  link="base_${suffix}"/>
-    </joint>
     <joint name="baselink_${suffix}_joint" type="floating">
       <origin rpy="0 0 0" xyz="0 0 0"/>
-      <parent link="base_${suffix}"/>
+      <parent link="${parent}"/>
       <child  link="baselink_${suffix}"/>
     </joint>
@@ -21,9 +14,4 @@
       <child  link="sensor_${suffix}"/>
     </joint>
-    <joint name="odom_${suffix}_joint" type="floating">
-      <origin rpy="0 0 0" xyz="0 0 0"/>
-      <parent link="baselink_${suffix}"/>
-      <child  link="odom_${suffix}"/>
-    </joint>
   </xacro:macro>
 </robot>

File: ros2/pybullet_ros/urdf/mas.urdf.xacro (robot description, xacro)
@@ -3,5 +3,5 @@
   <link name="map" />
   <link name="world"/>
-  <joint name="map_wolrd" type="fixed">
+  <joint name="map_world" type="fixed">
     <origin rpy="0 0 0" xyz="1 0 0"/>
     <parent link="map"/>
@@ -9,7 +9,7 @@
   </joint>
   <xacro:include filename="$(find pybullet_ros)/urdf/drone.urdf.xacro" />
-  <xacro:drone_macro suffix='a' parent='world' x_dist="0.3" y_dist="0.0" z_dist="1.0" radius="0" />
-  <xacro:drone_macro suffix='b' parent='world' x_dist="0.3" y_dist="0.6" z_dist="1.0" radius="0" />
-  <xacro:drone_macro suffix='c' parent='world' x_dist="-0.3" y_dist="0.0" z_dist="1.0" radius="0" />
-  <xacro:drone_macro suffix='d' parent='world' x_dist="-0.3" y_dist="0.6" z_dist="1.0" radius="0" />
+  <xacro:drone_macro suffix='a' parent='world' />
+  <xacro:drone_macro suffix='b' parent='world' />
+  <xacro:drone_macro suffix='c' parent='world' />
+  <xacro:drone_macro suffix='d' parent='world' />
 </robot>
